Commit message: change XX.p22 to p22_XX

File: p22_vehicle_description/urdf/vehicle.xacro (robot description, xacro)
@@ -2,5 +2,5 @@
 <robot xmlns:xacro="http://ros.org/wiki/xacro">
   <!-- load parameter -->
-  <xacro:property name="vehicle_info" value="${xacro.load_yaml('$(find vehicle_description.p22)/config/vehicle_info.param.yaml')}"/>
+  <xacro:property name="vehicle_info" value="${xacro.load_yaml('$(find p22_vehicle_description)/config/vehicle_info.param.yaml')}"/>
   <!-- vehicle body -->
   <link name="base_link">
@@ -8,5 +8,5 @@
       <origin xyz="${vehicle_info['/**']['ros__parameters']['wheel_base']/2.0} 0 0" rpy="${pi/2.0} 0 ${pi}"/>
       <geometry>
-        <mesh filename="package://vehicle_description.p22/mesh/vehicle.p22.fbx" scale="1 1 1"/>
+        <mesh filename="package://p22_vehicle_description/mesh/p22_vehicle.fbx" scale="1 1 1"/>
       </geometry>
     </visual>

Commit message: New Model Update!

File: p22_vehicle_description/urdf/vehicle.xacro (robot description, xacro)
@@ -6,7 +6,7 @@
   <link name="base_link">
     <visual>
-      <origin xyz="${vehicle_info['/**']['ros__parameters']['wheel_base']/2.0} 0 0" rpy="${pi/2.0} 0 ${pi}"/>
+      <origin xyz="0 0 0" rpy="${pi/2.0} 0 ${pi/2.0}"/>
       <geometry>
-        <mesh filename="package://p22_vehicle_description/mesh/p22_vehicle.fbx" scale="1 1 1"/>
+        <mesh filename="package://p22_vehicle_description/mesh/p22_vehicle.fbx" scale="0.01 0.01 0.01"/>
       </geometry>
     </visual>

Commit message: fix config & vehicle.xacro

File: p22_vehicle_description/urdf/vehicle.xacro (robot description, xacro)
@@ -6,5 +6,5 @@
   <link name="base_link">
     <visual>
-      <origin xyz="0 0 0" rpy="${pi/2.0} 0 ${pi/2.0}"/>
+      <origin xyz="0 0 0.17" rpy="${pi/2.0} 0 ${pi}"/>
       <geometry>
         <mesh filename="package://p22_vehicle_description/mesh/p22_vehicle.fbx" scale="0.01 0.01 0.01"/>
